File: Hardware Schematics/Electrical Schematics/Final Design/Final Design.kicad_sch (KiCad schematic)
At the start: 35 parts, among them J1 USB_C_Receptacle_PowerOnly_6P, SW1 SW_DPST, SW2 SW_DPST, SW3 SW_SPDT_MSM, SW4 SW_SPDT_MSM, SW5 SW_SPST, U1 Generic 48-24V Buck Converter, U2 Generic 24-5V Buck Converter, U4 Generic 1S LiPO Charger

Commit message: update circuit diagram to include discharge test setup
Other:
- added sheet Discharge Circuit (discharge.kicad_sch)
Changed lines of the file:
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@@
+		)
+	)
+	(sheet
+		(at 198.12 128.27)
+		(size 83.82 34.29)
+		(exclude_from_sim no)
+		(in_bom yes)
+		(on_board yes)
+		(dnp no)
+		(fields_autoplaced yes)
+		(stroke
+			(width 0.1524)
+			(type solid)
+		)
+		(fill
+			(color 0 0 0 0)
+		)
+		(property "Sheetname" "Discharge Circuit"
+			(at 198.12 127.5584 0)
+			(show_name no)
+			(do_not_autoplace no)
+			(effects
+				(font
+					(size 1.27 1.27)
+				)
+				(justify left bottom)
+			)
+		)
+		(property "Sheetfile" "discharge.kicad_sch"
+			(at 198.12 163.1446 0)
+			(show_name no)
+			(do_not_autoplace no)
+			(effects
+				(font
+					(size 1.27 1.27)
+				)
+				(justify left top)
+			)
+		)
+		(instances
+			(project "Final Design"
+				(path "/8a457180-428a-419a-bd41-bb68223cdc26"
+					(page "2")
+				)
+			)
 		)
 	)

Commit message: added missing fuse for battery terminal and seperate sensor diagrams
Parts:
- added F2, F3: 100A, symbol Device:Fuse
Connections:
- net Batt1_48V: now also F2.2; no longer BT1.1 (+)
- net Batt2_48V: now also F3.2; no longer BT3.1 (+)
- new net: BT3.1 (+), F3.1
- new net: BT1.1 (+), F2.1
Other:
- added sheet final_setup_no_sensor (final_setup_no_sensor.kicad_sch)
- moved on the sheet: SW3, SW4, U1, U2
